File: _autosave-unnamed-arisu52.kicad_pcb (KiCad board)
At the start: 2 copper layers, 376.6 x 95.8 mm, 129 parts, among them J1 Conn_01x04_Female, SW1 SW_Push, U1 ATmega32U4-M, Y1 Crystal_GND24_Small

Commit message: laid out diodes with respect to the switches
Parts:
- D24, D25, D26, D27, D39, D40, D41, D42, D52, D53, D8: moved to B.Cu
- moved D42 225.4 mm to (275.0, 136.5), turned to 102 degrees
- moved D53 217.7 mm to (279.8, 156.5), turned to 102 degrees
- moved D52 217.3 mm to (239.4, 163.5), turned to 102 degrees
- moved D27 213.3 mm to (280.4, 115.9), turned to 102 degrees
- moved D41 210.6 mm to (256.4, 140.4), turned to 102 degrees
- moved D40 197.1 mm to (237.7, 144.4), turned to 102 degrees
- moved D26 187.1 mm to (261.7, 119.8), turned to 102 degrees
- moved D39 179.7 mm to (219.1, 148.4), turned to 102 degrees
- moved D25 166.7 mm to (243.1, 123.8), turned to 102 degrees
- moved D24 162.8 mm to (224.5, 127.8), turned to 102 degrees
- moved D8 156.1 mm to (215.9, 110.1), turned to 102 degrees
- moved Y1 139.9 mm to (210.2, 75.4)
