File: unnamed-arisu52.kicad_pcb (KiCad board)
At the start: 2 copper layers, 376.6 x 95.8 mm, 129 parts, among them J1 Conn_01x04_Female, SW1 SW_Push, U1 ATmega32U4-M, Y1 Crystal_GND24_Small

Commit message: routed the matrix
Parts:
- D24, D25, D26, D27, D39, D40, D41, D42, D52, D53, D8, J1, U1: moved to B.Cu
- moved C3 271.5 mm to (167.3, 73.0)
- moved C7 271.5 mm to (161.5, 76.4)
- moved C9 271.5 mm to (161.5, 78.9)
- moved D42 223.4 mm to (272.3, 136.4), turned to 102 degrees
- moved D53 216.0 mm to (277.1, 156.3), turned to 102 degrees
- moved D52 215.7 mm to (236.7, 163.4), turned to 102 degrees
- moved D27 213.7 mm to (277.6, 115.7), turned to 102 degrees
- moved D41 208.8 mm to (253.6, 140.3), turned to 102 degrees
- moved D40 195.5 mm to (235.0, 144.3), turned to 102 degrees
- moved D26 185.3 mm to (259.0, 119.7), turned to 102 degrees
- moved D39 179.0 mm to (216.4, 148.2), turned to 102 degrees
- moved D25 165.5 mm to (240.4, 123.7), turned to 102 degrees
- moved D24 161.6 mm to (221.7, 127.6), turned to 102 degrees
- moved D8 154.8 mm to (213.1, 110.0), turned to 102 degrees
- moved J1 141.4 mm to (210.7, 54.0)
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Routing:
- net /ROW-2: track 0.00 -> 374.1 mm
- net /ROW-1: track 0.00 -> 361.8 mm
- net /ROW-3: track 0.00 -> 333.7 mm
- net /ROW-0: track 0.00 -> 330.3 mm
- net /COL-13: track 0.00 -> 82.6 mm
- net /COL-14: track 0.00 -> 69.4 mm
- net /COL-15: track 0.00 -> 67.8 mm
- net /COL-10: track 0.00 -> 66.0 mm
- net /COL-6: track 0.00 -> 65.4 mm
- net /COL-1: track 0.00 -> 65.0 mm
- net /COL-3: track 0.00 -> 64.7 mm
- net /COL-8: track 0.00 -> 63.9 mm
- net /COL-5: track 0.00 -> 63.5 mm
- net /COL-11: track 0.00 -> 44.9 mm
- net /COL-12: track 0.00 -> 44.1 mm
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Other:
- outline, holes or cut-outs redrawn
