File: unnamed-arisu52.kicad_pcb (KiCad board)
At the start: 2 copper layers, 376.6 x 95.8 mm, 129 parts, among them J1 Conn_01x04_Female, SW1 SW_Push, U1 ATmega32U4-M, Y1 Crystal_GND24_Small

Commit message: bro i dont know what this commit is maybe the last commit
Routing:
- net /ROW-1: track 585.1 -> 586.9 mm, vias 0 -> 2
- added copper zone on B.Cu, net GND
- added copper zone on F.Cu, net GND
Changed lines of the file:
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@@
   (segment (start 35.8775 107.3785) (end 35.8775 112.0785) (width 0.25) (layer "B.Cu") (net 22))
   (segment (start 35.8775 112.0785) (end 39.1795 115.3805) (width 0.25) (layer "B.Cu") (net 22))
+  (segment (start 392.888751 108.2675) (end 392.888751 116.629) (width 0.25) (layer "F.Cu") (net 23))
+  (segment (start 392.4935 104.7115) (end 392.888751 105.106751) (width 0.25) (layer "F.Cu") (net 23))
+  (segment (start 392.888751 116.629) (end 393.163251 116.9035) (width 0.25) (layer "F.Cu") (net 23))
+  (segment (start 392.888751 105.106751) (end 392.888751 108.2675) (width 0.25) (layer "F.Cu") (net 23))
+  (via (at 393.163251 116.9035) (size 0.8) (drill 0.4) (layers "F.Cu" "B.Cu") (net 23))
+  (via (at 392.4935 104.7115) (size 0.8) (drill 0.4) (layers "F.Cu" "B.Cu") (net 23))
   (segment (start 69.52325 118.6655) (end 69.53825 118.6805) (width 0.25) (layer "B.Cu") (net 23))
   (segment (start 100.49825 118.6805) (end 118.487976 118.6805) (width 0.25) (layer "B.Cu") (net 23))
+  (segment (start 391.386251 118.6805) (end 387.18825 118.6805) (width 0.25) (layer "B.Cu") (net 23))
   (segment (start 118.487976 118.6805) (end 119.576987 119.769511) (width 0.25) (layer "B.Cu") (net 23))
   (segment (start 263.292519 117.356511) (end 259.331801 121.317229) (width 0.25) (layer "B.Cu") (net 23))
   (segment (start 138.210699 123.730229) (end 152.883693 123.730229) (width 0.25) (layer "B.Cu") (net 23))
+  (segment (start 388.378424 100.596424) (end 392.4935 104.7115) (width 0.25) (layer "B.Cu") (net 23))
   (segment (start 193.70733 129.286) (end 193.754665 129.238665) (width 0.25) (layer "B.Cu") (net 23))
   (segment (start 255.511576 100.596424) (end 251.550858 104.557142) (width 0.25) (layer "B.Cu") (net 23))
@@
   (segment (start 348.440501 117.544499) (end 347.3045 118.6805) (width 0.25) (layer "B.Cu") (net 23))
   (segment (start 347.3045 118.6805) (end 346.168499 117.544499) (width 0.25) (layer "B.Cu") (net 23))
+  (segment (start 393.163251 116.9035) (end 391.386251 118.6805) (width 0.25) (layer "B.Cu") (net 23))
   (segment (start 69.53825 118.6805) (end 100.49825 118.6805) (width 0.25) (layer "B.Cu") (net 23))
   (segment (start 217.97067 108.51786) (end 208.46809 118.02044) (width 0.25) (layer "B.Cu") (net 23))
   (segment (start 119.576987 119.769511) (end 134.249981 119.769511) (width 0.25) (layer "B.Cu") (net 23))
   (segment (start 244.658807 121.317229) (end 240.698089 125.277947) (width 0.25) (layer "B.Cu") (net 23))
-  (segment (start 387.18825 118.6805) (end 389.3195 118.6805) (width 0.25) (layer "B.Cu") (net 23))
-  (segment (start 389.3195 118.6805) (end 392.43 115.57) (width 0.25) (layer "B.Cu") (net 23))
-  (segment (start 392.43 115.57) (end 392.43 104.648) (width 0.25) (layer "B.Cu") (net 23))
   (segment (start 200.02248 119.04744) (end 198.79588 119.04744) (width 0.25) (layer "B.Cu") (net 23))
   (segment (start 134.249981 119.769511) (end 138.210699 123.730229) (width 0.25) (layer "B.Cu") (net 23))
@@
   (segment (start 279.289502 118.6805) (end 277.965513 117.356511) (width 0.25) (layer "B.Cu") (net 23))
   (segment (start 387.18825 118.6805) (end 386.052249 117.544499) (width 0.25) (layer "B.Cu") (net 23))
-  (segment (start 392.43 104.648) (end 388.378424 100.596424) (width 0.25) (layer "B.Cu") (net 23))
   (segment (start 193.754665 129.238665) (end 222.064377 129.238665) (width 0.25) (layer "B.Cu") (net 23))
   (segment (start 208.46809 118.02044) (end 201.04948 118.02044) (width 0.25) (layer "B.Cu") (net 23))
@@
   (segment (start 194.564 97.93244) (end 193.871 97.23944) (width 0.25) (layer "B.Cu") (net 93))
   (segment (start 197.456547 125.88344) (end 201.327983 125.88344) (width 0.25) (layer "B.Cu") (net 93))
+  (zone (net 1) (net_name "GND") (layers F&B.Cu) (hatch edge 0.508)
+    (connect_pads yes (clearance 0.508))
+    (min_thickness 0.254) (filled_areas_thickness no)
+    (fill yes (thermal_gap 0.508) (thermal_bridge_width 0.508))
+    (polygon
+      (pts
+        (xy 398.7165 82.2325)
+        (xy 399.9865 130.7465)
+        (xy 398.7165 165.9255)
+        (xy 398.3355 173.0375)
+        (xy 201.6125 207.8355)
+        (xy 15.5575 178.2445)
+        (xy 14.4145 81.3435)
+      )
+    )
+  )
 )
